File: Hardware/KiCad Project/Antimatter-Control-Board/IMU.kicad_sch (KiCad schematic)
At the start: 8 parts, among them IC1 IIS2MDCTR

Commit message: Add power sheet and fix some ERC issues
Parts:
- AC1: footprint LSM6DS3USTR -> SamacSys_Parts:LSM6DS3USTR
- IC1: footprint IIS2MDCTR -> SamacSys_Parts:IIS2MDCTR
- R1, R2: footprint (none) -> Resistor_SMD:R_0201_0603Metric
Changed lines of the file:
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@@
 			)
 		)
-		(property "Footprint" ""
+		(property "Footprint" "Resistor_SMD:R_0201_0603Metric"
 			(at 105.41 157.48 0)
 			(effects
@@
 			)
 		)
-		(property "Footprint" "LSM6DS3USTR"
+		(property "Footprint" "SamacSys_Parts:LSM6DS3USTR"
 			(at 111.76 173.66 0)
 			(effects
@@
 			)
 		)
-		(property "Footprint" ""
+		(property "Footprint" "Resistor_SMD:R_0201_0603Metric"
 			(at 114.3 157.48 0)
 			(effects
@@
 			)
 		)
-		(property "Footprint" "IIS2MDCTR"
+		(property "Footprint" "SamacSys_Parts:IIS2MDCTR"
 			(at 234.95 188.9 0)
 			(effects
