File: Hardware/KiCad Project/Antimatter-Control-Board/Antimatter-Control-Board.kicad_sch (KiCad schematic)
At the start: 0 parts

Commit message: Connect up MCU
Other:
- sheet IMU & MAG ports: added IMU INT, MAG INT; removed IMUINT, MAGINT
- sheet MCU ports: added BATT SENSE, IMU INT, M1 IN1, M1 IN2, M2 IN1, M2 IN2, MAG INT, SCL, SDA; removed none
- sheet Power ports: added BATT SENSE; removed none
Changed lines of the file:
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@@
 		(company "Marc Rouillard")
 	)
+	(wire
+		(pts
+			(xy 151.13 95.25) (xy 151.13 115.57)
+		)
+		(stroke
+			(width 0)
+			(type default)
+		)
+	)
+	(wire
+		(pts
+			(xy 93.98 69.85) (xy 132.08 69.85)
+		)
+		(stroke
+			(width 0)
+			(type default)
+		)
+	)
+	(wire
+		(pts
+			(xy 175.26 81.28) (xy 198.12 81.28)
+		)
+		(stroke
+			(width 0)
+			(type default)
+		)
+	)
+	(wire
+		(pts
+			(xy 175.26 62.23) (xy 198.12 62.23)
+		)
+		(stroke
+			(width 0)
+			(type default)
+		)
+	)
+	(wire
+		(pts
+			(xy 156.21 95.25) (xy 156.21 115.57)
+		)
+		(stroke
+			(width 0)
+			(type default)
+		)
+	)
+	(wire
+		(pts
+			(xy 175.26 83.82) (xy 198.12 83.82)
+		)
+		(stroke
+			(width 0)
+			(type default)
+		)
+	)
+	(wire
+		(pts
+			(xy 153.67 95.25) (xy 153.67 115.57)
+		)
+		(stroke
+			(width 0)
+			(type default)
+		)
+	)
+	(wire
+		(pts
+			(xy 158.75 95.25) (xy 158.75 115.57)
+		)
+		(stroke
+			(width 0)
+			(type default)
+		)
+	)
+	(wire
+		(pts
+			(xy 175.26 64.77) (xy 198.12 64.77)
+		)
+		(stroke
+			(width 0)
+			(type default)
+		)
+	)
 	(sheet
-		(at 205.74 45.72)
+		(at 143.002 115.57)
 		(size 24.384 22.352)
 		(exclude_from_sim no)
@@
 		(on_board yes)
 		(dnp no)
-		(fields_autoplaced yes)
 		(stroke
 			(width 0.1524)
@@
 		)
 		(property "Sheetname" "IMU & MAG"
-			(at 205.74 45.0084 0)
+			(at 138.684 114.808 0)
 			(effects
 				(font
@@
 		)
 		(property "Sheetfile" "IMU.kicad_sch"
-			(at 205.74 68.6566 0)
+			(at 143.002 138.5066 0)
 			(effects
 				(font
@@
 			)
 		)
-		(pin "MAGINT" output
-			(at 205.74 62.23 180)
-			(effects
-				(font
-					(size 1.27 1.27)
-				)
-				(justify left)
-			)
-		)
-		(pin "IMUINT" output
-			(at 205.74 58.42 180)
-			(effects
-				(font
-					(size 1.27 1.27)
-				)
-				(justify left)
+		(pin "MAG INT" output
+			(at 158.75 115.57 90)
+			(effects
+				(font
+					(size 1.27 1.27)
+				)
+				(justify right)
+			)
+		)
+		(pin "IMU INT" output
+			(at 156.21 115.57 90)
+			(effects
+				(font
+					(size 1.27 1.27)
+				)
+				(justify right)
 			)
 		)
 		(pin "SDA" bidirectional
-			(at 205.74 50.8 180)
-			(effects
-				(font
-					(size 1.27 1.27)
-				)
-				(justify left)
+			(at 151.13 115.57 90)
+			(effects
+				(font
+					(size 1.27 1.27)
+				)
+				(justify right)
 			)
 		)
 		(pin "SCL" bidirectional
-			(at 205.74 54.61 180)
-			(effects
-				(font
-					(size 1.27 1.27)
-				)
-				(justify left)
+			(at 153.67 115.57 90)
+			(effects
+				(font
+					(size 1.27 1.27)
+				)
+				(justify right)
 			)
 		)
@@
 	)
 	(sheet
-		(at 217.678 124.206)
-		(size 21.336 11.43)
+		(at 198.12 77.47)
+		(size 21.082 10.16)
 		(exclude_from_sim no)
 		(in_bom yes)
@@
 		)
 		(property "Sheetname" "Motor Driver 2"
-			(at 217.678 123.4944 0)
+			(at 198.12 76.7584 0)
 			(effects
 				(font
@@
 		)
 		(property "Sheetfile" "Motor Driver 1.kicad_sch"
-			(at 217.678 136.2206 0)
+			(at 198.12 88.2146 0)
 			(effects
 				(font
@@
 		)
 		(pin "MOTOR REVERSE" input
-			(at 217.678 132.588 180)
+			(at 198.12 83.82 180)
 			(effects
 				(font
@@
 		)
 		(pin "MOTOR FORWARD" input
-			(at 217.678 127.508 180)
+			(at 198.12 81.28 180)
 			(effects
 				(font
@@
 	)
 	(sheet
-		(at 130.556 72.136)
+		(at 132.08 54.356)
 		(size 43.18 40.894)
 		(exclude_from_sim no)
@@
 		(on_board yes)
 		(dnp no)
-		(fields_autoplaced yes)
 		(stroke
 			(width 0.1524)
@@
 		)
 		(property "Sheetname" "MCU"
-			(at 130.556 71.4244 0)
+			(at 132.08 53.6444 0)
 			(effects
 				(font
@@
 		)
 		(property "Sheetfile" "MCU.kicad_sch"
-			(at 130.556 113.6146 0)
+			(at 156.21 52.07 0)
 			(effects
 				(font
@@
 				)
 				(justify left top)
+			)
+		)
+		(pin "IMU INT" input
+			(at 156.21 95.25 270)
+			(effects
+				(font
+					(size 1.27 1.27)
+				)
+				(justify left)
+			)
+		)
+		(pin "M1 IN1" output
+			(at 175.26 62.23 0)
+			(effects
+				(font
+					(size 1.27 1.27)
+				)
+				(justify right)
+			)
+		)
+		(pin "SCL" bidirectional
+			(at 153.67 95.25 270)
+			(effects
+				(font
+					(size 1.27 1.27)
+				)
+				(justify left)
+			)
+		)
+		(pin "M2 IN2" output
+			(at 175.26 83.82 0)
+			(effects
+				(font
+					(size 1.27 1.27)
+				)
+				(justify right)
+			)
+		)
+		(pin "M2 IN1" output
+			(at 175.26 81.28 0)
+			(effects
+				(font
+					(size 1.27 1.27)
+				)
+				(justify right)
+			)
+		)
+		(pin "BATT SENSE" passive
+			(at 132.08 69.85 180)
+			(effects
+				(font
+					(size 1.27 1.27)
+				)
+				(justify left)
+			)
+		)
+		(pin "M1 IN2" output
+			(at 175.26 64.77 0)
+			(effects
+				(font
+					(size 1.27 1.27)
+				)
+				(justify right)
+			)
+		)
+		(pin "SDA" bidirectional
+			(at 151.13 95.25 270)
+			(effects
+				(font
+					(size 1.27 1.27)
+				)
+				(justify left)
+			)
+		)
+		(pin "MAG INT" input
+			(at 158.75 95.25 270)
+			(effects
+				(font
+					(size 1.27 1.27)
+				)
+				(justify left)
 			)
 		)
@@
 	)
 	(sheet
-		(at 218.186 104.902)
+		(at 198.12 57.912)
 		(size 21.336 11.176)
 		(exclude_from_sim no)
@@
 		)
 		(property "Sheetname" "Motor Driver 1"
-			(at 218.186 104.1904 0)
+			(at 198.12 57.2004 0)
 			(effects
 				(font
@@
 		)
 		(property "Sheetfile" "Motor Driver 1.kicad_sch"
-			(at 218.186 116.6626 0)
+			(at 198.12 69.6726 0)
 			(effects
 				(font
@@
 		)
 		(pin "MOTOR REVERSE" input
-			(at 218.186 113.284 180)
+			(at 198.12 64.77 180)
 			(effects
 				(font
@@
 		)
 		(pin "MOTOR FORWARD" input
-			(at 218.186 108.204 180)
+			(at 198.12 62.23 180)
 			(effects
 				(font
@@
 	)
 	(sheet
-		(at 20.32 20.828)
+		(at 69.85 62.738)
 		(size 24.13 24.13)
 		(exclude_from_sim no)
@@
 		)
 		(property "Sheetname" "Power"
-			(at 20.32 20.1164 0)
+			(at 69.85 62.0264 0)
 			(effects
 				(font
@@
 		)
 		(property "Sheetfile" "Power.kicad_sch"
-			(at 20.32 45.5426 0)
+			(at 69.85 87.4526 0)
 			(effects
 				(font
@@
 			)
 		)
+		(pin "BATT SENSE" passive
+			(at 93.98 69.85 0)
+			(effects
+				(font
+					(size 1.27 1.27)
+				)
+				(justify right)
+			)
+		)
