File: Hardware/KiCad Project/Antimatter-Control-Board/MCU.kicad_sch (KiCad schematic)
At the start: 0 parts

Commit message: Change from nRF25832 to nRF25833 and copy reference schematic from datasheet
Parts:
- added AE1: 50 OHM CHIP ANTENNA, symbol Device:Antenna_Chip
- added C1, C2: 12pF, symbol Device:C_Small
- added C10: 100pF, symbol Device:C_Small
- added C11, C5, C7: 100nF, symbol Device:C_Small
- added C12, C13: 1uF, symbol Device:C_Small
- added C3: 1pF, symbol Device:C_Small
- added C4: 1.2pF, symbol Device:C_Small
- added C6: 4.7uF, symbol Device:C_Small
- added C9: N.C., symbol Device:C_Small
- added L1: 4.7nH, symbol Device:L_Small
- added L2: 2.2nH, symbol Device:L_Small
- added U3: nRF52833_QDxx, Package_DFN_QFN:QFN-40-1EP_5x5mm_P0.4mm_EP3.6x3.6mm, symbol MCU_Nordic:nRF52833_QDxx
- added X1: 32MHz, symbol Device:Crystal
Connections:
- new net: C1.1, U3.28 (XC1), X1.1
- new net: C2.1, U3.29 (XC2), X1.2
- new net: C13.1, C9.1, U3.26 (DEC6), U3.38 (DEC4)
- new net: AE1.2 (PCB_Trace), L2.2
- new net: C5.1, U3.1 (DEC1)
- new net: C3.1, L1.1, U3.24 (ANT)
- new net: C10.1, U3.27 (DEC3)
- new net: C4.1, L1.2, L2.1
- new net +3V3: C11.1, C12.1, C6.1, C7.1, U3.18 (VDD), U3.30 (VDD), U3.40 (VDD), U3.8 (VDD), U3.9 (VDDH)
- new net GND: AE1.1 (FEED), C1.2, C10.2, C11.2, C12.2, C13.2, C2.2, C3.2, C4.2, C5.2, C6.2, C7.2, C9.2, U3.10 (VBUS), U3.25 (VSS_PA), U3.37 (VSS), U3.41 (VSS)
- no-connect marks 0 -> 5
Other:
- note added: "RADIO CRYSTAL"

Commit message: Connect up MCU
Parts:
- added D2: LED, LED_SMD:LED_0603_1608Metric, symbol Device:LED
- added R6: 330, symbol Device:R_Small_US
Connections:
- net GND: now also R6.2
- net IMU INT: now reaches U3.14 (P0.15)
- net MAG INT: now reaches U3.15 (P0.17)
- net at U3.17 (P0.20): now also D2.2 (A)
- net BATT MONITOR: now reaches U3.32 (AIN0/P0.02)
- net M1 IN1: now reaches U3.33 (AIN4/P0.28)
- net M1 IN2: now reaches U3.34 (AIN5/P0.29)
- net M2 IN1: now reaches U3.35 (AIN6/P0.30)
- net M2 IN2: now reaches U3.36 (AIN7/P0.31)
- net SDA: now reaches U3.4 (AIN2/P0.04)
- net SCL: now reaches U3.5 (AIN3/P0.05)
- new net: D2.1 (K), R6.1
Other:
- note added: "ANTENNA & MATCHING"
- note added: "STATUS LED"
